Commit message: 添加仿真传感器

File: ros2_sim_ws/src/urdf_description/urdf/fishbot/actuator/caster.urdf.xacro (robot description, xacro)
@@ -45,4 +45,12 @@
             <!-- 围绕y轴旋转 -->
         </joint>
+        <gazebo reference="${caster_name}_link">
+            <material>Gazebo/Black</material>
+            <!-- 摩擦力 -->
+            <mu1 value="0"/>
+            <mu2 value="0"/>
+            <kp value="1000000000.0"/>
+            <kd value="1.0"/>
+        </gazebo>
     </xacro:macro>
 </robot>

File: ros2_sim_ws/src/urdf_description/urdf/fishbot/actuator/wheel.urdf.xacro (robot description, xacro)
@@ -45,4 +45,12 @@
             <axis xyz="0.0 1 0.0"/>
         </joint>
+        <gazebo reference="${wheel_name}_link">
+            <!-- <material>Gazebo/Black</material> -->
+            <!-- 摩擦力 -->
+            <mu1 value="20"/>
+            <mu2 value="20"/>
+            <kp value="1000000000.0"/>
+            <kd value="1.0"/>
+        </gazebo>
     </xacro:macro>
 </robot>

File: ros2_sim_ws/src/urdf_description/urdf/fishbot/fishbot.urdf.xacro (robot description, xacro)
@@ -10,4 +10,7 @@
 <xacro:include filename="$(find urdf_description)/urdf/fishbot/actuator/wheel.urdf.xacro" />
 <xacro:include filename="$(find urdf_description)/urdf/fishbot/actuator/caster.urdf.xacro" />
+<!-- 插件 -->
+<xacro:include filename="$(find urdf_description)/urdf/fishbot/plugins/gazebo_control_plugin.xacro" />
+<xacro:include filename="$(find urdf_description)/urdf/fishbot/plugins/gazebo_sensor_plugin.xacro" />
 <xacro:base_xacro length="0.12" radius="0.1"/>
 <xacro:imu_xacro xyz="0.0 0.0 0.02" />
@@ -18,3 +21,5 @@
 <xacro:caster_xacro caster_name="front_caster" xyz="0.08 0.0 -0.076" />
 <xacro:caster_xacro caster_name="back_caster" xyz="-0.08 0.0 -0.076" />
+<xacro:gazebo_control_plugin  />
+<xacro:gazebo_sensor_plugin  />
 </robot>

File: ros2_sim_ws/src/urdf_description/urdf/fishbot/sensor/camera.urdf.xacro (robot description, xacro)
@@ -34,4 +34,5 @@
             <xacro:box_inertia m="0.1" w="0.02" h="0.10" d="0.02" />
         </link>
+        <link name="camera_optical_link"></link>
         <!-- 定义关节 -->
         <joint name="camera_joint" type="fixed">
@@ -43,4 +44,13 @@
             <origin xyz="${xyz}" rpy="0 0 0" />
         </joint>
+        <!-- 定义关节 -->
+        <joint name="camera_optical_joint" type="fixed">
+            <!-- 关节连接的父链接 -->
+            <parent link="camera_link" />
+            <!-- 关节连接的子链接 -->
+            <child link="camera_optical_link" />
+            <!-- 关节的位置和旋转 -->
+            <origin xyz="0 0 0" rpy="${-pi/2} 0 ${-pi/2}" />
+        </joint>
     </xacro:macro>
 </robot>

File: ros2_sim_ws/src/urdf_description/urdf/fishbot/sensor/laser.urdf.xacro (robot description, xacro)
@@ -82,4 +82,10 @@
             <origin xyz="${xyz}" rpy="0 0 0" />
         </joint>
+        <gazebo reference="laser_link">
+            <material>Gazebo/Black</material>
+        </gazebo>
+        <gazebo reference="laser_cylinder_link">
+            <material>Gazebo/Black</material>
+        </gazebo>
     </xacro:macro>
 </robot>
